File: hardware/Big Ben Ornament.sch (KiCad schematic (older format))
At the start: 47 parts, among them IC1 23LC1024-I_P, J1 Conn_01x24_Female, Q1 Si1308EDL, SW1 SW_Push, SW2 SW_Push, SW3 SW_Push, SW4 SW_SPDT, U1 ATmega328P-AU, U2 TPS62203DBV, U3 DS3231M

Commit message: Commit prep
Parts:
- C5: value C -> 10u
- C7: value C -> 4u7
- R8: value R_US -> 62
Changed lines of the file:
@@
 P 3650 6950
 F 0 "C7" H 3765 6996 50  0000 L CNN
-F 1 "C" H 3765 6905 50  0000 L CNN
+F 1 "4u7" H 3765 6905 50  0000 L CNN
 F 2 "Capacitor_SMD:C_0805_2012Metric_Pad1.18x1.45mm_HandSolder" H 3688 6800 50  0001 C CNN
 F 3 "~" H 3650 6950 50  0001 C CNN
@@
 P 5200 6900
 F 0 "C5" H 5315 6946 50  0000 L CNN
-F 1 "C" H 5315 6855 50  0000 L CNN
+F 1 "10u" H 5315 6855 50  0000 L CNN
 F 2 "Capacitor_SMD:C_0805_2012Metric_Pad1.18x1.45mm_HandSolder" H 5238 6750 50  0001 C CNN
 F 3 "~" H 5200 6900 50  0001 C CNN
@@
 P 3850 4150
 F 0 "R8" V 3645 4150 50  0000 C CNN
-F 1 "R_US" V 3736 4150 50  0000 C CNN
+F 1 "62" V 3736 4150 50  0000 C CNN
 F 2 "Resistor_SMD:R_0805_2012Metric_Pad1.20x1.40mm_HandSolder" V 3890 4140 50  0001 C CNN
 F 3 "~" H 3850 4150 50  0001 C CNN
