File: hardware/Big Ben Ornament.kicad_pcb (KiCad board)
At the start: 4 copper layers, 32.5 x 138.7 mm, 51 parts, among them IC1 23LC1024-I_P, J1 Conn_01x24_Female, Q1 Si1308EDL, SW1 SW_Push, SW2 SW_Push, SW3 SW_Push, SW4 SW_SPDT, U1 ATmega328P-AU, U2 TPS62203DBV, U3 DS3231M

Commit message: added HTML BOM
Parts:
- C5: value C -> 10u
- C7: value C -> 4u7
- R8: value R_US -> 62
